File: PCBWorkshopSimple.kicad_sch (KiCad schematic)
At the start: 6 parts, among them J1 Neopixel, J2 I2C, J4 Connections, U2 WeMos_D1_mini

Commit message: Final touches
Parts:
- J2: footprint Connector_PinHeader_2.00mm:PinHeader_1x04_P2.00mm_Vertical -> Connector_PinHeader_2.54mm:PinHeader_1x04_P2.54mm_Vertical
Connections:
- net ANDRIS_SPEZIAL: now reaches J4.4 (Pin_4), U2.6 (MOSI/D7)
Changed lines of the file:
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@@
     (stroke (width 0) (type default) (color 0 0 0 0))
+  )
+  (label "ANDRIS_SPEZIAL" (at 136.398 89.662 0)
+    (effects (font (size 1.27 1.27)) (justify left bottom))
   )
   (global_label "LED" (shape input) (at 133.096 82.042 0) (fields_autoplaced)
@@
     (property "Reference" "J2" (id 0) (at 187.452 50.8 0))
     (property "Value" "I2C" (id 1) (at 187.452 53.34 0))
-    (property "Footprint" "Connector_PinHeader_2.00mm:PinHeader_1x04_P2.00mm_Vertical" (id 2) (at 187.452 62.738 0)
+    (property "Footprint" "Connector_PinHeader_2.54mm:PinHeader_1x04_P2.54mm_Vertical" (id 2) (at 187.452 62.738 0)
       (effects (font (size 1.27 1.27)) hide)
     )
@@
     )
     (path "/a51f058c-ae9e-4d69-8e71-d5af26dc99b2"
-      (reference "J2") (unit 1) (value "I2C") (footprint "Connector_PinHeader_2.00mm:PinHeader_1x04_P2.00mm_Vertical")
+      (reference "J2") (unit 1) (value "I2C") (footprint "Connector_PinHeader_2.54mm:PinHeader_1x04_P2.54mm_Vertical")
     )
     (path "/b197f5cc-8f5d-43bb-8a76-f5df2cd86ed2"
