File: PCBWorkshopSimple.kicad_pcb (KiCad board)
At the start: 2 copper layers, 44 x 27.4 mm, 6 parts, among them J1 Neopixel, J2 I2C, J4 Connections, U2 WeMos_D1_mini

Commit message: Final touches
Changed lines of the file:
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@@
     (fp_line (start 6.96 1.25) (end 6.96 -1.25) (layer "F.Fab") (width 0.1))
     (fp_line (start 6.96 -1.25) (end 0.66 -1.25) (layer "F.Fab") (width 0.1))
-    (pad "1" thru_hole circle (at 0 0 270) (size 1.6 1.6) (drill 0.8) (layers *.Cu *.Mask)
+    (pad "1" thru_hole oval (at 0 0 270) (size 3 2.5) (drill 0.8) (layers *.Cu *.Mask)
       (net 10 "Net-(D1-Pad1)") (pintype "passive"))
     (pad "2" thru_hole oval (at 7.62 0 270) (size 1.6 1.6) (drill 0.8) (layers *.Cu *.Mask)
@@
     (fp_arc (start -1.23 -1.469694) (mid 4.17 0.000016) (end -1.230016 1.469666) (layer "F.Fab") (width 0.1))
     (fp_circle (center 1.27 0) (end 3.77 0) (layer "F.Fab") (width 0.1) (fill none))
-    (pad "1" thru_hole rect (at 0 0 180) (size 1.8 1.8) (drill 0.9) (layers *.Cu *.Mask)
+    (pad "1" thru_hole oval (at 0 0 270) (size 3 2.5) (drill 0.9) (layers *.Cu *.Mask)
       (net 10 "Net-(D1-Pad1)") (pinfunction "K") (pintype "passive"))
-    (pad "2" thru_hole circle (at 2.54 0 180) (size 1.8 1.8) (drill 0.9) (layers *.Cu *.Mask)
+    (pad "2" thru_hole oval (at 2.54 0 270) (size 3 2.5) (drill 0.9) (layers *.Cu *.Mask)
       (net 11 "LED") (pinfunction "A") (pintype "passive"))
     (model "${KICAD6_3DMODEL_DIR}/LED_THT.3dshapes/LED_D5.0mm.wrl"

Commit message: Upload plot files
Other:
- board text removed: "TODO: - Check Groove I2C adapter orientation"
Changed lines of the file:
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@@
     (pad "6" thru_hole oval (at 0 12.7 180) (size 3 2) (drill 1) (layers *.Cu *.Mask)
       (net 15 "Net-(J4-Pad6)") (pinfunction "Pin_6") (pintype "passive"))
-    (pad "7" thru_hole oval (at 0 15.24 180) (size 3 2) (drill 1) (layers *.Cu *.Mask)
+    (pad "7" thru_hole oval (at 0 15.24 180) (size 3 2) (drill 0.8) (layers *.Cu *.Mask)
       (net 16 "Net-(J4-Pad7)") (pinfunction "Pin_7") (pintype "passive"))
     (model "${KICAD6_3DMODEL_DIR}/Connector_PinHeader_2.54mm.3dshapes/PinHeader_1x07_P2.54mm_Vertical.wrl"
@@
     (fp_line (start 6.96 1.25) (end 6.96 -1.25) (layer "F.Fab") (width 0.1))
     (fp_line (start 6.96 -1.25) (end 0.66 -1.25) (layer "F.Fab") (width 0.1))
-    (pad "1" thru_hole oval (at 0 0 270) (size 3 2.5) (drill 0.8) (layers *.Cu *.Mask)
+    (pad "1" thru_hole oval (at 0 0 270) (size 3 2.5) (drill 1) (layers *.Cu *.Mask)
       (net 10 "Net-(D1-Pad1)") (pintype "passive"))
-    (pad "2" thru_hole oval (at 7.62 0 270) (size 1.6 1.6) (drill 0.8) (layers *.Cu *.Mask)
+    (pad "2" thru_hole oval (at 7.62 0 270) (size 1.6 1.6) (drill 1) (layers *.Cu *.Mask)
       (net 1 "GND") (pintype "passive"))
     (model "${KICAD6_3DMODEL_DIR}/Resistor_THT.3dshapes/R_Axial_DIN0207_L6.3mm_D2.5mm_P7.62mm_Horizontal.wrl"
@@
     (fp_arc (start -1.23 -1.469694) (mid 4.17 0.000016) (end -1.230016 1.469666) (layer "F.Fab") (width 0.1))
     (fp_circle (center 1.27 0) (end 3.77 0) (layer "F.Fab") (width 0.1) (fill none))
-    (pad "1" thru_hole oval (at 0 0 270) (size 3 2.5) (drill 0.9) (layers *.Cu *.Mask)
+    (pad "1" thru_hole oval (at 0 0 270) (size 3 2.5) (drill 1) (layers *.Cu *.Mask)
       (net 10 "Net-(D1-Pad1)") (pinfunction "K") (pintype "passive"))
-    (pad "2" thru_hole oval (at 2.54 0 270) (size 3 2.5) (drill 0.9) (layers *.Cu *.Mask)
+    (pad "2" thru_hole oval (at 2.54 0 270) (size 3 2.5) (drill 1) (layers *.Cu *.Mask)
       (net 11 "LED") (pinfunction "A") (pintype "passive"))
     (model "${KICAD6_3DMODEL_DIR}/LED_THT.3dshapes/LED_D5.0mm.wrl"
@@
   )
   (gr_rect (start 114 66.6444) (end 158.0132 94.0348) (layer "Edge.Cuts") (width 0.1) (fill none))
-  (gr_text "TODO:\n\n- Check Groove I2C adapter orientation\n" (at 69 63) (layer "F.SilkS")
-    (effects (font (size 1 1) (thickness 0.15)) (justify left))
-  )
   (segment (start 147.386 79.06) (end 144.81 79.06) (width 0.8) (layer "B.Cu") (net 2))
   (segment (start 150.9268 82.6008) (end 147.386 79.06) (width 0.8) (layer "B.Cu") (net 2))
